Commit message: Without 2 bot in one

File: m2wr_description/urdf/follow.xacro (robot description, xacro)
@@ -1,5 +1,5 @@
 <?xml version="1.0" ?>
 <robot name="m2wr" xmlns:xacro="https://www.ros.org/wiki/xacro" >
-	<xacro:property name="cameraSize" value="0.05"/>
+  <xacro:property name="cameraSize" value="0.05"/>
   <xacro:property name="cameraMass" value="0.1"/>
   <material name="black">
@@ -28,5 +28,5 @@
   </material>
   <gazebo reference="link_chassis">
-    <material>Gazebo/Blue</material>
+    <material>Gazebo/black</material>
   </gazebo>
   <gazebo reference="link_left_wheel">
@@ -41,5 +41,5 @@
     <inertial>
       <mass value="5"/>
-      <origin rpy="0 0 0" xyz="0 0 0.1"/>
+      <origin rpy="0 0 0" xyz="8 10 0.1"/>
       <inertia ixx="0.0395416666667" ixy="0" ixz="0" iyy="0.106208333333" iyz="0" izz="0.106208333333"/>
     </inertial>
@@ -50,5 +50,5 @@
     </collision>
     <visual>
-      <origin rpy="0 0 0" xyz="0 0 0"/>
+      <origin rpy="0 0 0" xyz="8 10 0.0"/>
       <geometry>
         <box size="0.5 0.3 0.07"/>
@@ -58,5 +58,5 @@
     <!-- caster front -->
     <collision name="caster_front_collision">
-      <origin rpy=" 0 0 0" xyz="0.35 0 -0.05"/>
+      <origin rpy=" 0 0 0" xyz="8.35 10 -0.05"/>
       <geometry>
         <sphere radius="0.05"/>
@@ -74,5 +74,5 @@
     </collision>
     <visual name="caster_front_visual">
-      <origin rpy=" 0 0 0" xyz="0.2 0 -0.05"/>
+      <origin rpy=" 0 0 0" xyz="8.2 10 -0.05"/>
       <geometry>
         <sphere radius="0.05"/>
@@ -100,35 +100,7 @@
     </visual>
   </link>
-<!--Stick-->
-<link name="stick">
-    <!-- pose and inertial -->
-    <pose>0 0 0.1 0 0 0</pose>
-    <inertial>
-      <mass value="0.5"/>
-      <origin rpy="0 0 0" xyz="0 0 0.1"/>
-      <inertia ixx="0.00395416666667" ixy="0" ixz="0" iyy="0.0106208333333" iyz="0" izz="0.0106208333333"/>
-    </inertial>
-    <collision name="collision_chassis">
-      <geometry>
-        <box size="0.02 0.02 0.7"/>
-      </geometry>
-    </collision>
-    <visual>
-      <origin rpy="0 0 0" xyz="0 0 0"/>
-      <geometry>
-        <box size="0.02 0.02 0.7"/>
-      </geometry>
-      <material name="red"/>
-    </visual>
-</link>
- <!--   Joint for stick  -->
-  <joint name="joint_stick" type="fixed">
-    <origin rpy="0 0 0" xyz="0.0 0.0 0.38"/>
-    <child link="stick" />
-    <parent link="link_chassis"/>
-  </joint>
   <!--   Joint for right wheel  -->
   <joint name="joint_right_wheel" type="continuous">
-    <origin rpy="0 0 0" xyz="-0.05 0.15 0"/>
+    <origin rpy="0 0 0" xyz="7.95 10.15 0"/>
     <child link="link_right_wheel" />
     <parent link="link_chassis"/>
@@ -159,5 +131,5 @@
   <!--   Joint for right wheel  -->
   <joint name="joint_left_wheel" type="continuous">
-    <origin rpy="0 0 0" xyz="-0.05 -0.15 0"/>
+    <origin rpy="0 0 0" xyz="7.95 9.85 0"/>
     <child link="link_left_wheel" />
     <parent link="link_chassis"/>
@@ -175,71 +147,9 @@
       <wheelDiameter>0.2</wheelDiameter>
       <torque>0.1</torque>
-      <commandTopic>cmd_vel</commandTopic>
-      <odometryTopic>odom</odometryTopic>
-      <odometryFrame>odom</odometryFrame>
+      <commandTopic>cmd_vel1</commandTopic>
+      <odometryTopic>odom1</odometryTopic>
+      <odometryFrame>odom1</odometryFrame>
       <robotBaseFrame>link_chassis</robotBaseFrame>
     </plugin>
-  </gazebo>
- <link name="sensor_laser">
-    <inertial>
-      <origin xyz="0 0 0" rpy="0 0 0" />
-      <mass value="1" />
-      <!-- RANDOM INERTIA BELOW -->
-      <inertia ixx="0.02" ixy="0" ixz="0" iyy="0.02" iyz="0" izz="0.02"/>
-    </inertial>
-    <visual>
-      <origin xyz="0 0 0" rpy="0 0 0" />
-      <geometry>
-        <cylinder radius="0.05" length="0.1"/>
-      </geometry>
-      <material name="white" />
-    </visual>
-    <collision>
-      <origin xyz="0 0 0" rpy="0 0 0"/>
-      <geometry>
-        <cylinder radius="0.05" length="0.1"/>
-      </geometry>
-    </collision>
-  </link>
-  <joint name="joint_sensor_laser" type="fixed">
-    <origin xyz="0.15 0 0.05" rpy="0 0 0"/>
-    <parent link="link_chassis"/>
-    <child link="sensor_laser"/>
-  </joint>
-<xacro:macro name="cylinder_inertia" params="mass r l">
-    <inertia ixx="${mass*(3*r*r+l*l)/12}" ixy = "0" ixz = "0"
-                iyy="${mass*(3*r*r+l*l)/12}" iyz = "0" izz="${mass*(r*r)/2}" />
-</xacro:macro>
-<xacro:cylinder_inertia mass="1" r="0.05" l="0.1" />
-<gazebo reference="sensor_laser">
-    <sensor type="ray" name="head_hokuyo_sensor">
-      <pose>0 0 0 0 0 0</pose>
-      <visualize>false</visualize>
-      <update_rate>20</update_rate>
-      <ray>
-        <scan>
-          <horizontal>
-            <samples>720</samples>
-            <resolution>1</resolution>
-            <min_angle>-1.570796</min_angle>
-            <max_angle>1.570796</max_angle>
-          </horizontal>
-        </scan>
-        <range>
-          <min>0.10</min>
-          <max>10.0</max>
-          <resolution>0.01</resolution>
-        </range>
-        <noise>
-          <type>gaussian</type>
-          <mean>0.0</mean>
-          <stddev>0.01</stddev>
-        </noise>
-      </ray>
-      <plugin name="gazebo_ros_head_hokuyo_controller" filename="libgazebo_ros_laser.so">
-        <topicName>/m2wr/laser/scan</topicName>
-        <frameName>sensor_laser</frameName>
-      </plugin>
-    </sensor>
   </gazebo>
   <link name="camera">
@@ -265,7 +175,7 @@
   </link>
   <joint name="camera_joint" type="fixed">
-    <axis xyz="0.1 0 0.35" />
-    <origin xyz=".02 0 0.35" rpy="0 0 0"/>
-    <parent link="stick"/>
+    <axis xyz="1 0.0 0.0" />
+    <origin xyz="8.3 10.0 0" rpy="0 0 0"/>
+    <parent link="link_chassis"/>
     <child link="camera"/>
   </joint>
@@ -285,5 +195,5 @@
           <far>300</far>
         </clip>
-	<save enabled="true">
+  <save enabled="true">
       <path>mybot_gazebo/Images</path>
     </save>
@@ -292,5 +202,5 @@
         <alwaysOn>true</alwaysOn>
         <updateRate>0.0</updateRate>
-        <cameraName>mybot/camera1</cameraName>
+        <cameraName>mybot/camera2</cameraName>
         <imageTopicName>image_raw</imageTopicName>
         <cameraInfoTopicName>camera_info</cameraInfoTopicName>

Commit message: Files Added

File: m2wr_description/urdf/follow.xacro (robot description, xacro)
@@ -141,5 +141,5 @@
     <plugin filename="libgazebo_ros_diff_drive.so" name="differential_drive_controller">
       <alwaysOn>true</alwaysOn>
-      <updateRate>20</updateRate>
+      <updateRate>5</updateRate>
       <leftJoint>joint_left_wheel</leftJoint>
       <rightJoint>joint_right_wheel</rightJoint>
@@ -183,10 +183,10 @@
     <material>Gazebo/Green</material>
     <sensor type="camera" name="camera1">
-      <update_rate>30.0</update_rate>
+      <update_rate>5</update_rate>
       <camera name="head">
         <horizontal_fov>1.3962634</horizontal_fov>
         <image>
-          <width>800</width>
-          <height>800</height>
+          <width>400</width>
+          <height>400</height>
           <format>R8G8B8</format>
         </image>
@@ -195,11 +195,8 @@
           <far>300</far>
         </clip>
-  <save enabled="true">
-      <path>mybot_gazebo/Images</path>
-    </save>
       </camera>
       <plugin name="camera_controller" filename="libgazebo_ros_camera.so">
         <alwaysOn>true</alwaysOn>
-        <updateRate>0.0</updateRate>
+        <updateRate>5</updateRate>
         <cameraName>mybot/camera2</cameraName>
         <imageTopicName>image_raw</imageTopicName>

File: m2wr_description/urdf/m2wr.xacro (robot description, xacro)
@@ -1,5 +1,5 @@
 <?xml version="1.0" ?>
-<robot name="m2wr" xmlns:xacro="https://www.ros.org/wiki/xacro" >
-	<xacro:property name="cameraSize" value="0.05"/>
+<robot name="follow" xmlns:xacro="https://www.ros.org/wiki/xacro" >
+  <xacro:property name="cameraSize" value="0.05"/>
   <xacro:property name="cameraMass" value="0.1"/>
   <material name="black">
@@ -7,5 +7,5 @@
   </material>
   <material name="blue">
-    <color rgba="0.203125 0.23828125 0.28515625 1.0"/>
+    <color rgba="0.0 0.0 1.0 1.0"/>
   </material>
   <material name="green">
@@ -41,5 +41,5 @@
     <inertial>
       <mass value="5"/>
-      <origin rpy="0 0 0" xyz="0 0 0.1"/>
+      <origin rpy="0 0 0" xyz="8 8 0.1"/>
       <inertia ixx="0.0395416666667" ixy="0" ixz="0" iyy="0.106208333333" iyz="0" izz="0.106208333333"/>
     </inertial>
@@ -50,5 +50,5 @@
     </collision>
     <visual>
-      <origin rpy="0 0 0" xyz="0 0 0"/>
+      <origin rpy="0 0 0" xyz="8 8 0.0"/>
       <geometry>
         <box size="0.5 0.3 0.07"/>
@@ -58,5 +58,5 @@
     <!-- caster front -->
     <collision name="caster_front_collision">
-      <origin rpy=" 0 0 0" xyz="0.35 0 -0.05"/>
+      <origin rpy=" 0 0 0" xyz="8.35 8 -0.05"/>
       <geometry>
         <sphere radius="0.05"/>
@@ -74,5 +74,5 @@
     </collision>
     <visual name="caster_front_visual">
-      <origin rpy=" 0 0 0" xyz="0.2 0 -0.05"/>
+      <origin rpy=" 0 0 0" xyz="8.2 8 -0.05"/>
       <geometry>
         <sphere radius="0.05"/>
@@ -100,4 +100,42 @@
     </visual>
   </link>
+  <!--   Joint for right wheel  -->
+  <joint name="joint_right_wheel" type="continuous">
+    <origin rpy="0 0 0" xyz="7.95 8.15 0"/>
+    <child link="link_right_wheel" />
+    <parent link="link_chassis"/>
+    <axis rpy="0 0 0" xyz="0 1 0"/>
+    <limit effort="10000" velocity="1000"/>
+    <joint_properties damping="1.0" friction="1.0" />
+  </joint>
+  <!-- Left Wheel link -->
+  <link name="link_left_wheel">
+    <inertial>
+      <mass value="0.2"/>
+      <origin rpy="0 1.5707 1.5707" xyz="0 0 0"/>
+      <inertia ixx="0.00052666666" ixy="0" ixz="0" iyy="0.00052666666" iyz="0" izz="0.001"/>
+    </inertial>
+    <collision name="link_left_wheel_collision">
+      <origin rpy="0 1.5707 1.5707" xyz="0 0 0" />
+      <geometry>
+        <cylinder length="0.04" radius="0.1"/>
+      </geometry>
+    </collision>
+    <visual name="link_left_wheel_visual">
+      <origin rpy="0 1.5707 1.5707" xyz="0 0 0"/>
+      <geometry>
+        <cylinder length="0.04" radius="0.1"/>
+      </geometry>
+    </visual>
+  </link>
+  <!--   Joint for right wheel  -->
+  <joint name="joint_left_wheel" type="continuous">
+    <origin rpy="0 0 0" xyz="7.95 7.85 0"/>
+    <child link="link_left_wheel" />
+    <parent link="link_chassis"/>
+    <axis rpy="0 0 0" xyz="0 1 0"/>
+    <limit effort="10000" velocity="1000"/>
+    <joint_properties damping="1.0" friction="1.0" />
+  </joint>
 <!--Stick-->
 <link name="stick">
@@ -124,50 +162,12 @@
  <!--   Joint for stick  -->
   <joint name="joint_stick" type="fixed">
-    <origin rpy="0 0 0" xyz="0.0 0.0 0.38"/>
+    <origin rpy="0 0 0" xyz="8.0 8.0 0.30"/>
     <child link="stick" />
     <parent link="link_chassis"/>
   </joint>
-  <!--   Joint for right wheel  -->
-  <joint name="joint_right_wheel" type="continuous">
-    <origin rpy="0 0 0" xyz="-0.05 0.15 0"/>
-    <child link="link_right_wheel" />
-    <parent link="link_chassis"/>
-    <axis rpy="0 0 0" xyz="0 1 0"/>
-    <limit effort="10000" velocity="1000"/>
-    <joint_properties damping="1.0" friction="1.0" />
-  </joint>
-  <!-- Left Wheel link -->
-  <link name="link_left_wheel">
-    <inertial>
-      <mass value="0.2"/>
-      <origin rpy="0 1.5707 1.5707" xyz="0 0 0"/>
-      <inertia ixx="0.00052666666" ixy="0" ixz="0" iyy="0.00052666666" iyz="0" izz="0.001"/>
-    </inertial>
-    <collision name="link_left_wheel_collision">
-      <origin rpy="0 1.5707 1.5707" xyz="0 0 0" />
-      <geometry>
-        <cylinder length="0.04" radius="0.1"/>
-      </geometry>
-    </collision>
-    <visual name="link_left_wheel_visual">
-      <origin rpy="0 1.5707 1.5707" xyz="0 0 0"/>
-      <geometry>
-        <cylinder length="0.04" radius="0.1"/>
-      </geometry>
-    </visual>
-  </link>
-  <!--   Joint for right wheel  -->
-  <joint name="joint_left_wheel" type="continuous">
-    <origin rpy="0 0 0" xyz="-0.05 -0.15 0"/>
-    <child link="link_left_wheel" />
-    <parent link="link_chassis"/>
-    <axis rpy="0 0 0" xyz="0 1 0"/>
-    <limit effort="10000" velocity="1000"/>
-    <joint_properties damping="1.0" friction="1.0" />
-  </joint>
-  <gazebo>
+     <gazebo>
     <plugin filename="libgazebo_ros_diff_drive.so" name="differential_drive_controller">
       <alwaysOn>true</alwaysOn>
-      <updateRate>20</updateRate>
+      <updateRate>5</updateRate>
       <leftJoint>joint_left_wheel</leftJoint>
       <rightJoint>joint_right_wheel</rightJoint>
@@ -203,5 +203,5 @@
   </link>
   <joint name="joint_sensor_laser" type="fixed">
-    <origin xyz="0.15 0 0.05" rpy="0 0 0"/>
+    <origin xyz="8.15 8 0.05" rpy="0 0 0"/>
     <parent link="link_chassis"/>
     <child link="sensor_laser"/>
@@ -266,6 +266,6 @@
   <joint name="camera_joint" type="fixed">
     <axis xyz="0.1 0 0.35" />
-    <origin xyz=".02 0 0.35" rpy="0 0 0"/>
-    <parent link="stick"/>
+    <origin xyz="8.02 8 0.45" rpy="0 0 0"/>
+    <parent link="link_chassis"/>
     <child link="camera"/>
   </joint>
@@ -291,5 +291,5 @@
       <plugin name="camera_controller" filename="libgazebo_ros_camera.so">
         <alwaysOn>true</alwaysOn>
-        <updateRate>0.0</updateRate>
+        <updateRate>1</updateRate>
         <cameraName>mybot/camera1</cameraName>
         <imageTopicName>image_raw</imageTopicName>
