Commit message: Colour Changed

File: m2wr_description/urdf/m2wr.xacro (robot description, xacro)
@@ -26,11 +26,11 @@
   </material>
   <gazebo reference="link_chassis">
-    <material>Gazebo/Orange</material>
+    <material>Gazebo/Blue</material>
   </gazebo>
   <gazebo reference="link_left_wheel">
-    <material>Gazebo/Blue</material>
+    <material>Gazebo/Red</material>
   </gazebo>
   <gazebo reference="link_right_wheel">
-    <material>Gazebo/Blue</material>
+    <material>Gazebo/Red</material>
   </gazebo>
   <link name="link_chassis">

Commit message: 2 bot file

File: m2wr_description/urdf/m2wr.xacro (robot description, xacro)
@@ -105,5 +105,5 @@
     <pose>0 0 0.1 0 0 0</pose>
     <inertial>
-      <mass value="0.5"/>
+      <mass value="0.1"/>
       <origin rpy="0 0 0" xyz="0 0 0.1"/>
       <inertia ixx="0.00395416666667" ixy="0" ixz="0" iyy="0.0106208333333" iyz="0" izz="0.0106208333333"/>
@@ -273,10 +273,10 @@
     <material>Gazebo/Green</material>
     <sensor type="camera" name="camera1">
-      <update_rate>30.0</update_rate>
+      <update_rate>10.0</update_rate>
       <camera name="head">
         <horizontal_fov>1.3962634</horizontal_fov>
         <image>
-          <width>800</width>
-          <height>800</height>
+          <width>400</width>
+          <height>400</height>
           <format>R8G8B8</format>
         </image>

Commit message: Chnages in bot1_lane file

File: m2wr_description/urdf/m2wr.xacro (robot description, xacro)
@@ -162,5 +162,5 @@
  <!--   Joint for stick  -->
   <joint name="joint_stick" type="fixed">
-    <origin rpy="0 0 0" xyz="8.0 8.0 0.30"/>
+    <origin rpy="0 0 0" xyz="7.78 8 0.30"/>
     <child link="stick" />
     <parent link="link_chassis"/>
@@ -266,5 +266,5 @@
   <joint name="camera_joint" type="fixed">
     <axis xyz="0.1 0 0.35" />
-    <origin xyz="8.02 8 0.45" rpy="0 0 0"/>
+    <origin xyz="7.8 8 0.45" rpy="0 0 0"/>
     <parent link="link_chassis"/>
     <child link="camera"/>
@@ -273,5 +273,5 @@
     <material>Gazebo/Green</material>
     <sensor type="camera" name="camera1">
-      <update_rate>1</update_rate>
+      <update_rate>10</update_rate>
       <camera name="head">
         <horizontal_fov>1.3962634</horizontal_fov>
@@ -291,5 +291,5 @@
       <plugin name="camera_controller" filename="libgazebo_ros_camera.so">
         <alwaysOn>true</alwaysOn>
-        <updateRate>1</updateRate>
+        <updateRate>0</updateRate>
         <cameraName>mybot/camera1</cameraName>
         <imageTopicName>image_raw</imageTopicName>

Commit message: go.py added

File: m2wr_description/urdf/m2wr.xacro (robot description, xacro)
@@ -265,15 +265,15 @@
   </link>
   <joint name="camera_joint" type="fixed">
-    <axis xyz="0.1 0 0.35" />
-    <origin xyz="7.8 8 0.45" rpy="0 0 0"/>
+    <axis xyz="0.1 0 0.15" />
+    <origin xyz="7.8 8 0.45" rpy="0 0.0 0"/>
     <parent link="link_chassis"/>
     <child link="camera"/>
   </joint>
+  <!-- camera -->
   <gazebo reference="camera">
-    <material>Gazebo/Green</material>
     <sensor type="camera" name="camera1">
-      <update_rate>10</update_rate>
+      <update_rate>30.0</update_rate>
       <camera name="head">
-        <horizontal_fov>1.3962634</horizontal_fov>
+        <horizontal_fov>1.8</horizontal_fov>
         <image>
           <width>400</width>
@@ -285,15 +285,20 @@
           <far>300</far>
         </clip>
-	<save enabled="true">
-      <path>mybot_gazebo/Images</path>
-    </save>
+        <noise>
+          <type>gaussian</type>
+          <!-- Noise is sampled independently per pixel on each frame.
+               That pixel's noise value is added to each of its color
+               channels, which at that point lie in the range [0,1]. -->
+          <mean>0.0</mean>
+          <stddev>0.007</stddev>
+        </noise>
       </camera>
       <plugin name="camera_controller" filename="libgazebo_ros_camera.so">
         <alwaysOn>true</alwaysOn>
-        <updateRate>0</updateRate>
+        <updateRate>0.0</updateRate>
         <cameraName>mybot/camera1</cameraName>
         <imageTopicName>image_raw</imageTopicName>
         <cameraInfoTopicName>camera_info</cameraInfoTopicName>
-        <frameName>camera</frameName>
+        <frameName>camera_link</frameName>
         <hackBaseline>0.07</hackBaseline>
         <distortionK1>0.0</distortionK1>

Commit message: Hello

File: m2wr_description/urdf/m2wr.xacro (robot description, xacro)
@@ -162,5 +162,5 @@
  <!--   Joint for stick  -->
   <joint name="joint_stick" type="fixed">
-    <origin rpy="0 0 0" xyz="7.78 8 0.30"/>
+    <origin rpy="0 0 0" xyz="7.7 8 0.30"/>
     <child link="stick" />
     <parent link="link_chassis"/>
@@ -266,5 +266,5 @@
   <joint name="camera_joint" type="fixed">
     <axis xyz="0.1 0 0.15" />
-    <origin xyz="7.8 8 0.45" rpy="0 0.0 0"/>
+    <origin xyz="7.72 8 0.5" rpy="0 0.0 0"/>
     <parent link="link_chassis"/>
     <child link="camera"/>

Commit message: lane.py added

File: m2wr_description/urdf/m2wr.xacro (robot description, xacro)
@@ -162,5 +162,5 @@
  <!--   Joint for stick  -->
   <joint name="joint_stick" type="fixed">
-    <origin rpy="0 0 0" xyz="7.7 8 0.30"/>
+    <origin rpy="0 0 0" xyz="7.8 8 0.30"/>
     <child link="stick" />
     <parent link="link_chassis"/>
@@ -265,6 +265,6 @@
   </link>
   <joint name="camera_joint" type="fixed">
-    <axis xyz="0.1 0 0.15" />
-    <origin xyz="7.72 8 0.5" rpy="0 0.0 0"/>
+    <axis xyz="0.0 0 0.15" />
+    <origin xyz="7.82 8 0.5" rpy="0 0.0 0"/>
     <parent link="link_chassis"/>
     <child link="camera"/>
